File: microsd_basic.kicad_pcb (KiCad board)
At the start: 2 copper layers, 66.9 x 37.7 mm, 56 parts, among them Q1 BSS138PW,115, SW1 TS-1088-AR02016, SW2 TS-1088-AR02016, U1 AP2114HA-3.3TRG1, U2 TPS3823-33DBVR, U3 SI2301-ZE, U4 ESP32-S3-MINI-1

Commit message: Final v1.0
Parts:
- added 3.3V: TestPoint, TestPoint:TestPoint_Pad_D1.0mm, F.Cu at (167.8, 147.7)
- added 3.3V_SD: TestPoint, TestPoint:TestPoint_Pad_D1.0mm, F.Cu at (127.8, 134.0)
- added D+: TestPoint, TestPoint:TestPoint_Pad_D1.0mm, F.Cu at (145.7, 129.6)
- added D-: TestPoint, TestPoint:TestPoint_Pad_D1.0mm, F.Cu at (155.9, 128.3)
- added GND: TestPoint, TestPoint:TestPoint_Pad_D1.0mm, F.Cu at (137.1, 131.3)
- added TP8: TestPoint, TestPoint:TestPoint_Pad_D1.0mm, F.Cu at (127.6, 128.7)
- added VBUS: TestPoint, TestPoint:TestPoint_Pad_D1.0mm, F.Cu at (161.1, 127.0)
- moved R4 0.22 mm to (152.2, 129.6)
- moved D3 0.13 mm to (150.0, 129.3)
Routing:
- net /VBUS: track 8.99 -> 30.4 mm, vias 1 -> 3
- net /D-: track 4.45 -> 10.6 mm
- net +3.3V: track 146.9 -> 153.0 mm
- net /D+: track 4.90 -> 9.08 mm
- net /3.3V_SD: track 40.9 -> 44.1 mm
- net GND: track 103.2 -> 104.6 mm, vias 65 -> 66
