File: microsd_basic.kicad_sch (KiCad schematic)
At the start: 56 parts, among them Q1 BSS138PW,115, SW1 TS-1088-AR02016, SW2 TS-1088-AR02016, U1 AP2114HA-3.3TRG1, U2 TPS3823-33DBVR, U3 SI2301-ZE, U4 ESP32-S3-MINI-1

Commit message: Final v1.0
Parts:
- added TP1, TP2, TP3, TP4, TP6, TP7, TP8: TestPoint, TestPoint:TestPoint_Pad_D1.0mm, symbol Connector:TestPoint
Connections:
- net +3.3V: now also TP2.1, TP8.1
- net 3.3V_SD: now also TP4.1
- net D+: now also TP7.1
- net D-: now also TP6.1
- net GND: now also TP3.1
- net VBUS: now also TP1.1
Other:
- moved on the sheet: C6, R10
